File: PCB/usb-passwd.kicad_pcb (KiCad board)
At the start: 2 copper layers, 0 parts

Commit message: Netlist finished, started the layout
Parts:
- added C1: CSMALL, c_0805, B.Cu at (146.9, 103.0)
- added C2: CSMALL, c_0805, B.Cu at (147.6, 96.5)
- added C3: C, c_0805, F.Cu at (150.0, 102.4)
- added C4: C, c_0805, B.Cu at (161.2, 107.6)
- added D1: DBG, LED-0805, F.Cu at (175.0, 106.2)
- added D2: USER, LED-0805, F.Cu at (174.9, 109.6)
- added K1: UART, UART-POGO, F.Cu at (153.0, 113.4)
- added P1: ICSP, ICSP-POGO, F.Cu at (155.6, 100.8)
- added P2: USB, USB-A, F.Cu at (141.4, 108.2)
- added P3: SW1, SW-SMD, F.Cu at (169.2, 108.1)
- added P4: SW2, SW-SMD, F.Cu at (162.1, 108.1)
- added R1: R, SM0805, B.Cu at (175.0, 106.2)
- added R2: R, SM0805, B.Cu at (174.9, 109.5)
- added R3: R, SM0805, B.Cu at (147.1, 111.9)
- added U1: PIC18F14K50, SSOP-20-MCHIP, F.Cu at (153.2, 108.0)
- added X1: CRYSTAL-SMD, XTAL-SMD-UM, B.Cu at (147.1, 99.7)
Other:
- net class Default: clearance 0.254 -> 0.17; trace_width 0.254 -> 0.17
- rule trace_clearance: 0.254 -> 0.17
- rule trace_min: 0.254 -> 0.1524
- rule via_min_drill: 0.508 -> 0.3
- rule via_min_size: 0.889 -> 0.5
