File: PCB/usb-passwd.sch (KiCad schematic (older format))
At the start: 2 parts

Commit message: More schematics
Schematics partly done
Parts:
- removed P?: ICSP, ~, symbol CONN_6
- added C? (x2): CSMALL, ~, symbol CSMALL
- added C? (x2): C, ~, symbol C
- added D?: USER, ~, symbol LED
- added D?: DBG, ~, symbol LED
- added P?: DBG_UART, ~, symbol CONN_2
- added P?: SW1, ~, symbol CONN_2
- added P?: SW2, ~, symbol CONN_2
- added P?: ICSP, ~, symbol CONN_5
- added R?: R, ~, symbol R
- added U?: PIC18F14K50, ~, symbol PIC18F14K50
- added X?: CRYSTAL, ~, symbol CRYSTAL
Connections:
- net labels added: D+, D-, GND, OSC1, OSC2, PGC, PGD, UART_RX, UART_TX, Vcc, Vpp
- wire segments 0 -> 38
Other:
- note added: "Connectors"
- note added: "Oscillator"
- moved on the sheet: P?

Commit message: Schematics finished
Schematics are done
Parts:
- added R? (x2): R, ~, symbol R
Connections:
- net labels added: +5V, BUTTON1, BUTTON2, DBG_LED, USER_LED
- wire segments 38 -> 58
- no-connect marks 0 -> 6
Other:
- note added: "Power"
- note added: "User interface"
- moved on the sheet: C?, D?, P?, R?, U?, X?

Commit message: Netlist started
Parts:
- gave numbers to parts that had none: 16
Changed lines of the file:
@@
 $EndDescr
 $Comp
-L CONN_4 P?
+L CONN_4 P3
 U 1 1 55DE3238
 P 1250 6650
-F 0 "P?" V 1200 6650 50  0000 C CNN
+F 0 "P3" V 1200 6650 50  0000 C CNN
 F 1 "USB" V 1300 6650 50  0000 C CNN
 F 2 "~" H 1250 6650 60  0000 C CNN
@@
 $EndComp
 $Comp
-L PIC18F14K50 U?
+L PIC18F14K50 U1
 U 1 1 55EAE6AB
 P 7350 2900
-F 0 "U?" H 7250 2200 60  0000 C CNN
+F 0 "U1" H 7250 2200 60  0000 C CNN
 F 1 "PIC18F14K50" H 7350 3500 60  0000 C CNN
 F 2 "~" H 6850 3450 60  0000 C CNN
@@
 $EndComp
 $Comp
-L CONN_2 P?
+L CONN_2 P2
 U 1 1 55EAE7E0
 P 1250 5100
-F 0 "P?" V 1200 5100 40  0000 C CNN
+F 0 "P2" V 1200 5100 40  0000 C CNN
 F 1 "DBG_UART" V 1300 5100 40  0000 C CNN
 F 2 "~" H 1250 5100 60  0000 C CNN
@@
 $EndComp
 $Comp
-L CONN_2 P?
+L CONN_2 P4
 U 1 1 55EAE843
 P 2600 2000
-F 0 "P?" V 2550 2000 40  0000 C CNN
+F 0 "P4" V 2550 2000 40  0000 C CNN
 F 1 "SW1" V 2650 2000 40  0000 C CNN
 F 2 "~" H 2600 2000 60  0000 C CNN
@@
 $EndComp
 $Comp
-L CONN_2 P?
+L CONN_2 P5
 U 1 1 55EAE852
 P 2600 2400
-F 0 "P?" V 2550 2400 40  0000 C CNN
+F 0 "P5" V 2550 2400 40  0000 C CNN
 F 1 "SW2" V 2650 2400 40  0000 C CNN
 F 2 "~" H 2600 2400 60  0000 C CNN
@@
 $EndComp
 $Comp
-L LED D?
+L LED D2
 U 1 1 55EAE8DB
 P 2400 1600
-F 0 "D?" H 2400 1700 50  0000 C CNN
+F 0 "D2" H 2400 1700 50  0000 C CNN
 F 1 "USER" H 2400 1500 50  0000 C CNN
 F 2 "~" H 2400 1600 60  0000 C CNN
@@
 $EndComp
 $Comp
-L LED D?
+L LED D1
 U 1 1 55EAE8F2
 P 2400 1200
-F 0 "D?" H 2400 1300 50  0000 C CNN
+F 0 "D1" H 2400 1300 50  0000 C CNN
 F 1 "DBG" H 2400 1100 50  0000 C CNN
 F 2 "~" H 2400 1200 60  0000 C CNN
@@
 $EndComp
 $Comp
-L CRYSTAL X?
+L CRYSTAL X1
 U 1 1 55EAEA36
 P 1950 3650
-F 0 "X?" H 1950 3800 60  0000 C CNN
+F 0 "X1" H 1950 3800 60  0000 C CNN
 F 1 "CRYSTAL" H 1950 3500 60  0000 C CNN
 F 2 "~" H 1950 3650 60  0000 C CNN
@@
 $EndComp
 $Comp
-L CSMALL C?
+L CSMALL C1
 U 1 1 55EAFAA9
 P 1400 3550
-F 0 "C?" H 1425 3600 30  0000 L CNN
+F 0 "C1" H 1425 3600 30  0000 L CNN
 F 1 "CSMALL" H 1425 3500 30  0000 L CNN
 F 2 "~" H 1400 3550 60  0000 C CNN
@@
 $EndComp
 $Comp
-L CSMALL C?
+L CSMALL C2
 U 1 1 55EAFAB8
 P 2450 3550
-F 0 "C?" H 2475 3600 30  0000 L CNN
+F 0 "C2" H 2475 3600 30  0000 L CNN
 F 1 "CSMALL" H 2475 3500 30  0000 L CNN
 F 2 "~" H 2450 3550 60  0000 C CNN
@@
 $EndComp
 $Comp
-L C C?
+L C C3
 U 1 1 55EAFAD6
 P 6300 2150
-F 0 "C?" H 6300 2250 40  0000 L CNN
+F 0 "C3" H 6300 2250 40  0000 L CNN
 F 1 "C" H 6306 2065 40  0000 L CNN
 F 2 "~" H 6338 2000 30  0000 C CNN
@@
 $EndComp
 $Comp
-L R R?
+L R R3
 U 1 1 55EAFAE5
 P 5800 2100
-F 0 "R?" V 5880 2100 40  0000 C CNN
+F 0 "R3" V 5880 2100 40  0000 C CNN
 F 1 "R" V 5807 2101 40  0000 C CNN
 F 2 "~" V 5730 2100 30  0000 C CNN
@@
 $EndComp
 $Comp
-L C C?
+L C C4
 U 1 1 55EAFAF4
 P 8800 2100
-F 0 "C?" H 8800 2200 40  0000 L CNN
+F 0 "C4" H 8800 2200 40  0000 L CNN
 F 1 "C" H 8806 2015 40  0000 L CNN
 F 2 "~" H 8838 1950 30  0000 C CNN
@@
 Connection ~ 5800 2800
 $Comp
-L CONN_5 P?
+L CONN_5 P1
 U 1 1 55EB0049
 P 1200 5950
-F 0 "P?" V 1150 5950 50  0000 C CNN
+F 0 "P1" V 1150 5950 50  0000 C CNN
 F 1 "ICSP" V 1250 5950 50  0000 C CNN
 F 2 "~" H 1200 5950 60  0000 C CNN
@@
 GND
 $Comp
-L R R?
+L R R2
 U 1 1 55EB1D69
 P 1750 1600
-F 0 "R?" V 1830 1600 40  0000 C CNN
+F 0 "R2" V 1830 1600 40  0000 C CNN
 F 1 "R" V 1757 1601 40  0000 C CNN
 F 2 "~" V 1680 1600 30  0000 C CNN
@@
 $EndComp
 $Comp
-L R R?
+L R R1
 U 1 1 55EB1D78
 P 1750 1200
-F 0 "R?" V 1830 1200 40  0000 C CNN
+F 0 "R1" V 1830 1200 40  0000 C CNN
 F 1 "R" V 1757 1201 40  0000 C CNN
 F 2 "~" V 1680 1200 30  0000 C CNN
@@
 USER_LED
 $Comp
-L GND #PWR?
+L GND #PWR01
 U 1 1 55EB212B
 P 4500 6100
-F 0 "#PWR?" H 4500 6100 30  0001 C CNN
+F 0 "#PWR01" H 4500 6100 30  0001 C CNN
 F 1 "GND" H 4500 6030 30  0001 C CNN
 F 2 "" H 4500 6100 60  0000 C CNN
@@
 $EndComp
 $Comp
-L +5V #PWR?
+L +5V #PWR02
 U 1 1 55EB213A
 P 4000 6100
-F 0 "#PWR?" H 4000 6190 20  0001 C CNN
+F 0 "#PWR02" H 4000 6190 20  0001 C CNN
 F 1 "+5V" H 4000 6190 30  0000 C CNN
 F 2 "" H 4000 6100 60  0000 C CNN

Commit message: More netlist, footprint work
Added more stuff to netlist, created some footprints.
Parts:
- removed P2: DBG_UART, ~, symbol CONN_2
- added K1: UART, ~, symbol CONN_3
Connections:
- wire segments 58 -> 67
Changed lines of the file:
@@
 Sheet 1 1
 Title ""
-Date "5 sep 2015"
+Date "6 nov 2015"
 Rev ""
 Comp ""
@@
 $EndComp
 $Comp
-L CONN_2 P2
-U 1 1 55EAE7E0
-P 1250 5100
-F 0 "P2" V 1200 5100 40  0000 C CNN
-F 1 "DBG_UART" V 1300 5100 40  0000 C CNN
-F 2 "~" H 1250 5100 60  0000 C CNN
-F 3 "~" H 1250 5100 60  0000 C CNN
-	1    1250 5100
-	-1   0    0    1
-$EndComp
-$Comp
 L CONN_2 P4
 U 1 1 55EAE843
@@
 	1950 3100 1950 3300
 Wire Wire Line
-	1400 3300 2450 3300
+	1400 3300 1950 3300
+Wire Wire Line
+	1950 3300 2450 3300
 Wire Wire Line
 	2450 3300 2450 3450
@@
 OSC2
 Wire Wire Line
-	1600 5000 2100 5000
+	1600 5100 2100 5100
 Wire Wire Line
 	1600 5200 2100 5200
-Text Label 2100 5000 0    60   ~ 0
+Text Label 2100 5100 0    60   ~ 0
 UART_RX
 Text Label 2100 5200 0    60   ~ 0
@@
 	8400 2500 8400 1800
 Wire Wire Line
-	6300 1800 8800 1800
+	6300 1800 8400 1800
+Wire Wire Line
+	8400 1800 8600 1800
+Wire Wire Line
+	8600 1800 8800 1800
 Wire Wire Line
 	8600 1800 8600 1550
@@
 	6050 2500 6300 2500
 Wire Wire Line
-	6050 1700 6050 2500
+	6050 1700 6050 1850
+Wire Wire Line
+	6050 1850 6050 2500
 Text Label 6050 1700 0    60   ~ 0
 Vcc
@@
 	5800 2350 5800 2800
 Wire Wire Line
-	5500 2800 6300 2800
+	5500 2800 5800 2800
+Wire Wire Line
+	5800 2800 6300 2800
 Connection ~ 5800 2800
 $Comp
@@
 PGC
 Wire Wire Line
-	8400 2600 9600 2600
-Wire Wire Line
-	8400 2700 9600 2700
+	8400 2600 9250 2600
+Wire Wire Line
+	9250 2600 9600 2600
+Wire Wire Line
+	8400 2700 9400 2700
+Wire Wire Line
+	9400 2700 9600 2700
 Wire Wire Line
 	9250 2600 9250 2400
@@
 $EndComp
 Wire Wire Line
-	2600 1200 2600 1600
+	2600 1200 2600 1400
+Wire Wire Line
+	2600 1400 2600 1600
 Wire Wire Line
 	2600 1400 2700 1400
@@
 NoConn ~ 6300 3300
 NoConn ~ 8400 3100
+$Comp
+L CONN_3 K1
+U 1 1 563D0640
+P 1250 5100
+F 0 "K1" V 1200 5100 50  0000 C CNN
+F 1 "UART" V 1300 5100 40  0000 C CNN
+F 2 "~" H 1250 5100 60  0000 C CNN
+F 3 "~" H 1250 5100 60  0000 C CNN
+	1    1250 5100
+	-1   0    0    1
+$EndComp
+Wire Wire Line
+	1600 5000 2100 5000
+Text Label 2100 5000 0    60   ~ 0
+GND
 $EndSCHEMATC

Commit message: Netlist finished, started the layout
Parts:
- removed P4: SW1, ~, symbol CONN_2
- removed P5: SW2, ~, symbol CONN_2
- removed X1: CRYSTAL, ~, symbol CRYSTAL
- added P3: SW1, ~, symbol CONN_4
- added P4: SW2, ~, symbol CONN_4
- added X1: CRYSTAL-SMD, ~, symbol CRYSTAL-SMD
- renumbered P3 to P2
Connections:
- wire segments 67 -> 61
- no-connect marks 6 -> 10
Other:
- moved on the sheet: D1, D2, R1, R2
Changed lines of the file:
@@
 LIBS:remote_bt_shutter
 LIBS:imx23_phone
+LIBS:general_parts
 LIBS:usb-passwd-cache
 EELAYER 27 0
@@
 Sheet 1 1
 Title ""
-Date "6 nov 2015"
+Date "7 nov 2015"
 Rev ""
 Comp ""
@@
 $EndDescr
 $Comp
-L CONN_4 P3
+L CONN_4 P2
 U 1 1 55DE3238
 P 1250 6650
-F 0 "P3" V 1200 6650 50  0000 C CNN
+F 0 "P2" V 1200 6650 50  0000 C CNN
 F 1 "USB" V 1300 6650 50  0000 C CNN
 F 2 "~" H 1250 6650 60  0000 C CNN
@@
 $EndComp
 $Comp
-L CONN_2 P4
-U 1 1 55EAE843
-P 2600 2000
-F 0 "P4" V 2550 2000 40  0000 C CNN
-F 1 "SW1" V 2650 2000 40  0000 C CNN
-F 2 "~" H 2600 2000 60  0000 C CNN
-F 3 "~" H 2600 2000 60  0000 C CNN
-	1    2600 2000
-	1    0    0    -1
-$EndComp
-$Comp
-L CONN_2 P5
-U 1 1 55EAE852
-P 2600 2400
-F 0 "P5" V 2550 2400 40  0000 C CNN
-F 1 "SW2" V 2650 2400 40  0000 C CNN
-F 2 "~" H 2600 2400 60  0000 C CNN
-F 3 "~" H 2600 2400 60  0000 C CNN
-	1    2600 2400
-	1    0    0    -1
-$EndComp
-$Comp
 L LED D2
 U 1 1 55EAE8DB
-P 2400 1600
-F 0 "D2" H 2400 1700 50  0000 C CNN
-F 1 "USER" H 2400 1500 50  0000 C CNN
-F 2 "~" H 2400 1600 60  0000 C CNN
-F 3 "~" H 2400 1600 60  0000 C CNN
-	1    2400 1600
+P 2400 1500
+F 0 "D2" H 2400 1600 50  0000 C CNN
+F 1 "USER" H 2400 1400 50  0000 C CNN
+F 2 "~" H 2400 1500 60  0000 C CNN
+F 3 "~" H 2400 1500 60  0000 C CNN
+	1    2400 1500
 	1    0    0    -1
 $EndComp
@@
 L LED D1
 U 1 1 55EAE8F2
-P 2400 1200
-F 0 "D1" H 2400 1300 50  0000 C CNN
-F 1 "DBG" H 2400 1100 50  0000 C CNN
-F 2 "~" H 2400 1200 60  0000 C CNN
-F 3 "~" H 2400 1200 60  0000 C CNN
-	1    2400 1200
-	1    0    0    -1
-$EndComp
-$Comp
-L CRYSTAL X1
-U 1 1 55EAEA36
-P 1950 3650
-F 0 "X1" H 1950 3800 60  0000 C CNN
-F 1 "CRYSTAL" H 1950 3500 60  0000 C CNN
-F 2 "~" H 1950 3650 60  0000 C CNN
-F 3 "~" H 1950 3650 60  0000 C CNN
-	1    1950 3650
+P 2400 1100
+F 0 "D1" H 2400 1200 50  0000 C CNN
+F 1 "DBG" H 2400 1000 50  0000 C CNN
+F 2 "~" H 2400 1100 60  0000 C CNN
+F 3 "~" H 2400 1100 60  0000 C CNN
+	1    2400 1100
 	1    0    0    -1
 $EndComp
@@
 	1950 3100 1950 3300
 Wire Wire Line
-	1400 3300 1950 3300
-Wire Wire Line
-	1950 3300 2450 3300
+	1400 3300 2450 3300
 Wire Wire Line
 	2450 3300 2450 3450
@@
 	8400 2500 8400 1800
 Wire Wire Line
-	6300 1800 8400 1800
-Wire Wire Line
-	8400 1800 8600 1800
-Wire Wire Line
-	8600 1800 8800 1800
+	6300 1800 8800 1800
 Wire Wire Line
 	8600 1800 8600 1550
@@
 	6050 2500 6300 2500
 Wire Wire Line
-	6050 1700 6050 1850
-Wire Wire Line
-	6050 1850 6050 2500
+	6050 1700 6050 2500
 Text Label 6050 1700 0    60   ~ 0
 Vcc
@@
 	5800 2350 5800 2800
 Wire Wire Line
-	5500 2800 5800 2800
-Wire Wire Line
-	5800 2800 6300 2800
+	5500 2800 6300 2800
 Connection ~ 5800 2800
 $Comp
@@
 PGC
 Wire Wire Line
-	8400 2600 9250 2600
-Wire Wire Line
-	9250 2600 9600 2600
-Wire Wire Line
-	8400 2700 9400 2700
-Wire Wire Line
-	9400 2700 9600 2700
+	8400 2600 9600 2600
+Wire Wire Line
+	8400 2700 9600 2700
 Wire Wire Line
 	9250 2600 9250 2400
@@
 Text Label 1300 1900 2    60   ~ 0
 BUTTON1
-Text Label 1300 2300 2    60   ~ 0
+Text Label 1300 2450 2    60   ~ 0
 BUTTON2
 Wire Wire Line
-	2250 1900 1300 1900
-Wire Wire Line
-	2250 2300 1300 2300
-Wire Wire Line
-	2250 2100 1300 2100
-Wire Wire Line
-	2250 2500 1300 2500
+	1300 1900 2250 1900
+Wire Wire Line
+	1300 2450 2250 2450
+Wire Wire Line
+	1300 2100 2250 2100
+Wire Wire Line
+	1300 2650 2250 2650
 Text Label 1300 2100 2    60   ~ 0
 GND
-Text Label 1300 2500 2    60   ~ 0
+Text Label 1300 2650 2    60   ~ 0
 GND
 $Comp
 L R R2
 U 1 1 55EB1D69
-P 1750 1600
-F 0 "R2" V 1830 1600 40  0000 C CNN
-F 1 "R" V 1757 1601 40  0000 C CNN
-F 2 "~" V 1680 1600 30  0000 C CNN
-F 3 "~" H 1750 1600 30  0000 C CNN
-	1    1750 1600
+P 1750 1500
+F 0 "R2" V 1830 1500 40  0000 C CNN
+F 1 "R" V 1757 1501 40  0000 C CNN
+F 2 "~" V 1680 1500 30  0000 C CNN
+F 3 "~" H 1750 1500 30  0000 C CNN
+	1    1750 1500
 	0    -1   -1   0
 $EndComp
@@
 L R R1
 U 1 1 55EB1D78
-P 1750 1200
-F 0 "R1" V 1830 1200 40  0000 C CNN
-F 1 "R" V 1757 1201 40  0000 C CNN
-F 2 "~" V 1680 1200 30  0000 C CNN
-F 3 "~" H 1750 1200 30  0000 C CNN
-	1    1750 1200
+P 1750 1100
+F 0 "R1" V 1830 1100 40  0000 C CNN
+F 1 "R" V 1757 1101 40  0000 C CNN
+F 2 "~" V 1680 1100 30  0000 C CNN
+F 3 "~" H 1750 1100 30  0000 C CNN
+	1    1750 1100
 	0    -1   -1   0
 $EndComp
 Wire Wire Line
-	2600 1200 2600 1400
-Wire Wire Line
-	2600 1400 2600 1600
-Wire Wire Line
-	2600 1400 2700 1400
-Connection ~ 2600 1400
-Text Label 2700 1400 0    60   ~ 0
-GND
-Wire Wire Line
-	2200 1600 2000 1600
-Wire Wire Line
-	2000 1200 2200 1200
-Wire Wire Line
-	1500 1600 1300 1600
-Wire Wire Line
-	1500 1200 1300 1200
-Text Label 1300 1600 2    60   ~ 0
+	2600 1100 2600 1500
+Wire Wire Line
+	2600 1300 2700 1300
+Connection ~ 2600 1300
+Text Label 2700 1300 0    60   ~ 0
+GND
+Wire Wire Line
+	2200 1500 2000 1500
+Wire Wire Line
+	2000 1100 2200 1100
+Wire Wire Line
+	1500 1500 1300 1500
+Wire Wire Line
+	1500 1100 1300 1100
+Text Label 1300 1500 2    60   ~ 0
 USER_LED
-Text Label 1300 1200 2    60   ~ 0
+Text Label 1300 1100 2    60   ~ 0
 DBG_LED
 Wire Notes Line
@@
 USER_LED
 $Comp
-L GND #PWR01
+L GND #PWR2
 U 1 1 55EB212B
 P 4500 6100
-F 0 "#PWR01" H 4500 6100 30  0001 C CNN
+F 0 "#PWR2" H 4500 6100 30  0001 C CNN
 F 1 "GND" H 4500 6030 30  0001 C CNN
 F 2 "" H 4500 6100 60  0000 C CNN
@@
 $EndComp
 $Comp
-L +5V #PWR02
+L +5V #PWR1
 U 1 1 55EB213A
 P 4000 6100
-F 0 "#PWR02" H 4000 6190 20  0001 C CNN
+F 0 "#PWR1" H 4000 6190 20  0001 C CNN
 F 1 "+5V" H 4000 6190 30  0000 C CNN
 F 2 "" H 4000 6100 60  0000 C CNN
@@
 Text Label 2100 5000 0    60   ~ 0
 GND
+$Comp
+L CONN_4 P3
+U 1 1 563E5C65
+P 2600 2050
+F 0 "P3" V 2550 2050 50  0000 C CNN
+F 1 "SW1" V 2650 2050 50  0000 C CNN
+F 2 "~" H 2600 2050 60  0000 C CNN
+F 3 "~" H 2600 2050 60  0000 C CNN
+	1    2600 2050
+	1    0    0    -1
+$EndComp
+$Comp
+L CONN_4 P4
+U 1 1 563E5C74
+P 2600 2600
+F 0 "P4" V 2550 2600 50  0000 C CNN
+F 1 "SW2" V 2650 2600 50  0000 C CNN
+F 2 "~" H 2600 2600 60  0000 C CNN
+F 3 "~" H 2600 2600 60  0000 C CNN
+	1    2600 2600
+	1    0    0    -1
+$EndComp
+NoConn ~ 2250 2550
+NoConn ~ 2250 2750
+NoConn ~ 2250 2000
+NoConn ~ 2250 2200
+$Comp
+L CRYSTAL-SMD X1
+U 1 1 563E5E83
+P 1950 3650
+F 0 "X1" H 1950 3800 60  0000 C CNN
+F 1 "CRYSTAL-SMD" H 1950 3500 60  0000 C CNN
+F 2 "~" H 1950 3650 60  0000 C CNN
+F 3 "~" H 1950 3650 60  0000 C CNN
+	1    1950 3650
+	1    0    0    -1
+$EndComp
+Wire Wire Line
+	2250 3550 2250 3300
+Connection ~ 2250 3300
+Wire Wire Line
+	1650 3550 1650 3300
+Connection ~ 1650 3300
 $EndSCHEMATC
